File: mainboard.kicad_pcb (KiCad board)
At the start: 2 copper layers, 26 parts, among them U1 LIS2DW12, U2 AP2205-3.0, U3 BQ21080, U4 STM32L412KBTx

Commit message: Diode layout, majority of schema, tile thoughts
Parts:
- added C10: 100n, Capacitor_SMD:C_0402_1005Metric, F.Cu at (77.2, 162.1)
- added C11: 4p3, Capacitor_SMD:C_0402_1005Metric, F.Cu at (77.2, 164.1)
- added C12: 4p3, Capacitor_SMD:C_0402_1005Metric, F.Cu at (77.2, 166.0)
- added C8: 100n, Capacitor_SMD:C_0402_1005Metric, F.Cu at (77.2, 158.1)
- added C9: 100n, Capacitor_SMD:C_0402_1005Metric, F.Cu at (77.2, 160.1)
- added Q1: PMOS, Package_TO_SOT_SMD:SOT-23-3, F.Cu at (81.2, 159.4)
- added Q2: PMOS, Package_TO_SOT_SMD:SOT-23-3, F.Cu at (81.2, 163.8)
- added R5: 100k, Resistor_SMD:R_0402_1005Metric, F.Cu at (92.5, 158.2)
- added R6: 10k, Resistor_SMD:R_0402_1005Metric, F.Cu at (92.5, 160.1)
- added R7: 100k, Resistor_SMD:R_0402_1005Metric, F.Cu at (92.5, 162.1)
- added REF**: LED_WS2812B-2020_PLCC4_2.0x2.0mm, LED_SMD:LED_WS2812B-2020_PLCC4_2.0x2.0mm, F.Cu at (185.7, 78.0)
- added REF**: LED_WS2812B-2020_PLCC4_2.0x2.0mm, LED_SMD:LED_WS2812B-2020_PLCC4_2.0x2.0mm, B.Cu at (183.1, 104.1)
- added REF**1: LED_WS2812B-2020_PLCC4_2.0x2.0mm, LED_SMD:LED_WS2812B-2020_PLCC4_2.0x2.0mm, F.Cu at (180.6, 79.0)
- added REF**1: LED_WS2812B-2020_PLCC4_2.0x2.0mm, LED_SMD:LED_WS2812B-2020_PLCC4_2.0x2.0mm, B.Cu at (178.3, 102.2)
- added REF**10: LED_WS2812B-2020_PLCC4_2.0x2.0mm, LED_SMD:LED_WS2812B-2020_PLCC4_2.0x2.0mm, F.Cu at (195.0, 100.5)
- added REF**10: LED_WS2812B-2020_PLCC4_2.0x2.0mm, LED_SMD:LED_WS2812B-2020_PLCC4_2.0x2.0mm, B.Cu at (196.7, 83.8)
- added REF**11: LED_WS2812B-2020_PLCC4_2.0x2.0mm, LED_SMD:LED_WS2812B-2020_PLCC4_2.0x2.0mm, F.Cu at (197.9, 96.2)
- added REF**11: LED_WS2812B-2020_PLCC4_2.0x2.0mm, LED_SMD:LED_WS2812B-2020_PLCC4_2.0x2.0mm, B.Cu at (198.6, 88.6)
- added REF**12: LED_WS2812B-2020_PLCC4_2.0x2.0mm, LED_SMD:LED_WS2812B-2020_PLCC4_2.0x2.0mm, F.Cu at (198.9, 91.2)
- added REF**12: LED_WS2812B-2020_PLCC4_2.0x2.0mm, LED_SMD:LED_WS2812B-2020_PLCC4_2.0x2.0mm, B.Cu at (198.6, 93.8)
- added REF**13: LED_WS2812B-2020_PLCC4_2.0x2.0mm, LED_SMD:LED_WS2812B-2020_PLCC4_2.0x2.0mm, F.Cu at (197.9, 86.1)
- added REF**13: LED_WS2812B-2020_PLCC4_2.0x2.0mm, LED_SMD:LED_WS2812B-2020_PLCC4_2.0x2.0mm, B.Cu at (196.7, 98.5)
- added REF**14: LED_WS2812B-2020_PLCC4_2.0x2.0mm, LED_SMD:LED_WS2812B-2020_PLCC4_2.0x2.0mm, F.Cu at (195.0, 81.8)
- added REF**14: LED_WS2812B-2020_PLCC4_2.0x2.0mm, LED_SMD:LED_WS2812B-2020_PLCC4_2.0x2.0mm, B.Cu at (193.0, 102.2)
- added REF**15: LED_WS2812B-2020_PLCC4_2.0x2.0mm, LED_SMD:LED_WS2812B-2020_PLCC4_2.0x2.0mm, F.Cu at (190.7, 79.0)
- added REF**15: LED_WS2812B-2020_PLCC4_2.0x2.0mm, LED_SMD:LED_WS2812B-2020_PLCC4_2.0x2.0mm, B.Cu at (188.3, 104.1)
- added REF**2: LED_WS2812B-2020_PLCC4_2.0x2.0mm, LED_SMD:LED_WS2812B-2020_PLCC4_2.0x2.0mm, F.Cu at (176.3, 81.8)
- added REF**2: LED_WS2812B-2020_PLCC4_2.0x2.0mm, LED_SMD:LED_WS2812B-2020_PLCC4_2.0x2.0mm, B.Cu at (174.7, 98.5)
- added REF**3: LED_WS2812B-2020_PLCC4_2.0x2.0mm, LED_SMD:LED_WS2812B-2020_PLCC4_2.0x2.0mm, F.Cu at (173.5, 86.1)
- added REF**3: LED_WS2812B-2020_PLCC4_2.0x2.0mm, LED_SMD:LED_WS2812B-2020_PLCC4_2.0x2.0mm, B.Cu at (172.7, 93.8)
- added REF**4: LED_WS2812B-2020_PLCC4_2.0x2.0mm, LED_SMD:LED_WS2812B-2020_PLCC4_2.0x2.0mm, F.Cu at (172.5, 91.2)
- added REF**4: LED_WS2812B-2020_PLCC4_2.0x2.0mm, LED_SMD:LED_WS2812B-2020_PLCC4_2.0x2.0mm, B.Cu at (172.7, 88.6)
- added REF**5: LED_WS2812B-2020_PLCC4_2.0x2.0mm, LED_SMD:LED_WS2812B-2020_PLCC4_2.0x2.0mm, F.Cu at (173.5, 96.2)
- added REF**5: LED_WS2812B-2020_PLCC4_2.0x2.0mm, LED_SMD:LED_WS2812B-2020_PLCC4_2.0x2.0mm, B.Cu at (174.7, 83.8)
- added REF**6: LED_WS2812B-2020_PLCC4_2.0x2.0mm, LED_SMD:LED_WS2812B-2020_PLCC4_2.0x2.0mm, F.Cu at (176.3, 100.5)
- added REF**6: LED_WS2812B-2020_PLCC4_2.0x2.0mm, LED_SMD:LED_WS2812B-2020_PLCC4_2.0x2.0mm, B.Cu at (178.3, 80.2)
- added REF**7: LED_WS2812B-2020_PLCC4_2.0x2.0mm, LED_SMD:LED_WS2812B-2020_PLCC4_2.0x2.0mm, F.Cu at (180.6, 103.4)
- added REF**7: LED_WS2812B-2020_PLCC4_2.0x2.0mm, LED_SMD:LED_WS2812B-2020_PLCC4_2.0x2.0mm, B.Cu at (183.1, 78.2)
- added REF**8: LED_WS2812B-2020_PLCC4_2.0x2.0mm, LED_SMD:LED_WS2812B-2020_PLCC4_2.0x2.0mm, F.Cu at (185.7, 104.4)
- added REF**8: LED_WS2812B-2020_PLCC4_2.0x2.0mm, LED_SMD:LED_WS2812B-2020_PLCC4_2.0x2.0mm, B.Cu at (188.3, 78.2)
- added REF**9: LED_WS2812B-2020_PLCC4_2.0x2.0mm, LED_SMD:LED_WS2812B-2020_PLCC4_2.0x2.0mm, F.Cu at (190.7, 103.4)
- added REF**9: LED_WS2812B-2020_PLCC4_2.0x2.0mm, LED_SMD:LED_WS2812B-2020_PLCC4_2.0x2.0mm, B.Cu at (193.0, 80.2)
- added Y2: 32.768kHz, Crystal:Crystal_SMD_3215-2Pin_3.2x1.5mm, F.Cu at (166.4, 89.2)
- moved U4 77.7 mm to (185.7, 91.2)
Connections:
- U4 pad 10: unconnected-(U4-PA4-Pad10) -> LED IN
- U4 pad 12: unconnected-(U4-PA6-Pad12) -> LEDPowerCtrl
- U4 pad 13: unconnected-(U4-PA7-Pad13) -> BH1730PowerCtrl
- U4 pad 19: unconnected-(U4-PA9-Pad19) -> TX
- U4 pad 2: unconnected-(U4-PC14-Pad2) -> Net-(U4-PC14)
- U4 pad 20: unconnected-(U4-PA10-Pad20) -> RX
- U4 pad 23: unconnected-(U4-PA13-Pad23) -> SWDIO
- U4 pad 24: unconnected-(U4-PA14-Pad24) -> SWCLK
- U4 pad 29: unconnected-(U4-PB6-Pad29) -> SCL
- U4 pad 3: unconnected-(U4-PC15-Pad3) -> Net-(U4-PC15)
- U4 pad 30: unconnected-(U4-PB7-Pad30) -> SDA
- U4 pad 31: unconnected-(U4-PH3-Pad31) -> Net-(U4-PH3)
- U4 pad 4: unconnected-(U4-NRST-Pad4) -> Net-(U4-NRST)
- U4 pad 6: unconnected-(U4-PA0-Pad6) -> IMU_INT1
Other:
- board outline added: 124.2 x 261.1 mm

Commit message: Rev A layout. pending review
Parts:
- removed Q1: PMOS, Package_TO_SOT_SMD:SOT-23-3
- removed TP10: DIO, TestPoint:TestPoint_Pad_D1.0mm
- removed TP11: VBUS, TestPoint:TestPoint_Pad_D1.0mm
- removed TP7, TP8: GND, TestPoint:TestPoint_Pad_D1.0mm
- removed TP9: CLK, TestPoint:TestPoint_Pad_D1.0mm
- removed Y2: 32.768kHz, Crystal:Crystal_SMD_3215-2Pin_3.2x1.5mm
- added BT1: 200mAh, Components:battery_20x30, F.Cu at (185.7, 78.9)
- added C13: 100n, Capacitor_SMD:C_0402_1005Metric, F.Cu at (163.6, 95.5)
- added C14: 100n, Capacitor_SMD:C_0402_1005Metric, F.Cu at (172.3, 86.9)
- added C15: 100n, Capacitor_SMD:C_0402_1005Metric, F.Cu at (166.9, 85.5)
- added J1: Conn_01x04_Pin, Connector_PinHeader_2.54mm:PinHeader_1x04_P2.54mm_Vertical, F.Cu at (207.6, 87.5)
- added Q3: Q_PMOS_GSD, Package_TO_SOT_SMD:SOT-23, F.Cu at (177.8, 93.2)
- added U5: BH1730, Components:WSOF6, F.Cu at (180.7, 92.1)
- added Y1: 32.768k, Crystal:Crystal_SMD_3215-2Pin_3.2x1.5mm, F.Cu at (173.0, 83.4)
- Q2: value PMOS -> Q_PMOS_GSD; footprint Package_TO_SOT_SMD:SOT-23-3 -> Package_TO_SOT_SMD:SOT-23
- TP3, TP4: moved to B.Cu
- moved TP5 192.1 mm to (202.3, 100.7)
- moved TP6 186.0 mm to (197.0, 100.7)
- moved TP1 182.5 mm to (193.7, 87.2)
- moved TP2 182.5 mm to (193.7, 90.2)
- moved TP3 177.3 mm to (189.4, 89.4), turned to 180 degrees
- moved TP4 177.0 mm to (189.4, 91.4), turned to 180 degrees
- moved C3 167.3 mm to (185.7, 94.0), turned to 180 degrees
- moved C2 167.2 mm to (202.9, 98.4), turned to 0 degrees
- moved C4 166.4 mm to (185.7, 93.0), turned to 180 degrees
- moved U2 161.4 mm to (199.6, 98.4), turned to 180 degrees
- moved R1 160.4 mm to (188.3, 91.2), turned to 90 degrees
- moved C1 156.3 mm to (197.0, 98.3), turned to 90 degrees
- moved U1 155.8 mm to (185.7, 91.2), turned to -90 degrees
- moved R2 155.5 mm to (185.4, 86.6), turned to -90 degrees
- moved R4 153.9 mm to (203.1, 94.2), turned to 0 degrees
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Connections:
- C8 pad 1: +3V0 -> ALVCC
- C9 pad 1: +3V0 -> ALVCC
- Q2 pad 1: Net-(D1-VCC) -> LEDPowerCtrl
- Q2 pad 2: LEDP0werCtrl -> +BATT
- Q2 pad 3: +3V0 -> /LED_PWR
- R7 pad 1: +3V0 -> +BATT
- R7 pad 2: LEDP0werCtrl -> LEDPowerCtrl
- REF** pad 2: (no net) -> GND (x2)
- REF** pad 4: (no net) -> /LED_PWR (x2)
- REF**1 pad 2: (no net) -> GND (x2)
- REF**1 pad 4: (no net) -> /LED_PWR (x2)
- REF**10 pad 2: (no net) -> GND (x2)
- REF**10 pad 4: (no net) -> /LED_PWR (x2)
- REF**11 pad 2: (no net) -> GND (x2)
- REF**11 pad 4: (no net) -> /LED_PWR (x2)
- REF**12 pad 2: (no net) -> GND (x2)
- REF**12 pad 4: (no net) -> /LED_PWR (x2)
- REF**13 pad 2: (no net) -> GND (x2)
- REF**13 pad 4: (no net) -> /LED_PWR (x2)
- REF**14 pad 2: (no net) -> GND (x2)
- REF**14 pad 3: (no net) -> LED IN
- REF**14 pad 4: (no net) -> /LED_PWR (x2)
- REF**15 pad 2: (no net) -> GND (x2)
- REF**15 pad 4: (no net) -> /LED_PWR (x2)
- REF**2 pad 2: (no net) -> GND (x2)
- REF**2 pad 4: (no net) -> /LED_PWR (x2)
- REF**3 pad 2: (no net) -> GND (x2)
- REF**3 pad 4: (no net) -> /LED_PWR (x2)
- REF**4 pad 2: (no net) -> GND (x2)
- REF**4 pad 4: (no net) -> /LED_PWR (x2)
- REF**5 pad 2: (no net) -> GND (x2)
- REF**5 pad 4: (no net) -> /LED_PWR (x2)
- REF**6 pad 2: (no net) -> GND (x2)
- REF**6 pad 4: (no net) -> /LED_PWR (x2)
- REF**7 pad 4: (no net) -> /LED_PWR (x2)
- REF**7 pad 2: (no net) -> GND
- REF**8 pad 2: (no net) -> GND (x2)
- REF**8 pad 4: (no net) -> /LED_PWR (x2)
- REF**9 pad 2: (no net) -> GND (x2)
- REF**9 pad 4: (no net) -> /LED_PWR (x2)
- U4 pad 13: BH1730PowerCtrl -> unconnected-(U4-PA7-Pad13)
- U4 pad 25: unconnected-(U4-PA15-Pad25) -> BH1730PowerCtrl
Routing:
- net /LED_PWR: track 0.00 -> 187.4 mm, vias 0 -> 15
- net (no net): track 0.00 -> 172.3 mm, vias 0 -> 1
- net +3V0: track 0.00 -> 78.2 mm, vias 0 -> 5
- net SWDIO: track 0.00 -> 44.1 mm, vias 0 -> 2
- net +BATT: track 0.00 -> 43.6 mm, vias 0 -> 4
- net SWCLK: track 0.00 -> 41.8 mm, vias 0 -> 2
- net SDA: track 0.00 -> 40.3 mm, vias 0 -> 4
- net SCL: track 0.00 -> 37.6 mm
- net IMU_INT1: track 0.00 -> 26.6 mm, vias 0 -> 2
- net LEDPowerCtrl: track 0.00 -> 25.0 mm, vias 0 -> 2
- net LED IN: track 0.00 -> 14.5 mm
- net ALVCC: track 0.00 -> 9.88 mm, vias 0 -> 2
- net Net-(U4-PC15): track 0.00 -> 7.71 mm
- net VCC: track 0.00 -> 7.44 mm
- net GND: track 0.00 -> 6.63 mm, vias 0 -> 61
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- added copper zone on B.Cu, net GND
- added copper zone on F.Cu, net GND
Other:
- board size 124.2 x 261.1 mm -> 66 x 30 mm

Commit message: Rev 0 layout complete. ORdering as protoptype.
Parts:
- removed Q3: Q_PMOS_GSD, Package_TO_SOT_SMD:SOT-23
- added Q1: Q_PMOS_GSD, Package_TO_SOT_SMD:SOT-23, F.Cu at (177.5, 93.2)
- added R8: 100k, Resistor_SMD:R_0402_1005Metric, F.Cu at (175.0, 93.2)
- added R9: 100k, Resistor_SMD:R_0402_1005Metric, F.Cu at (178.3, 78.2)
- added REF**: TestPoint_Pad_D1.0mm, TestPoint:TestPoint_Pad_D1.0mm, B.Cu at (171.3, 77.5)
- added RX1: RX, TestPoint:TestPoint_Pad_D1.0mm, F.Cu at (167.9, 98.3)
- added TP10: 3v, TestPoint:TestPoint_Pad_D1.0mm, F.Cu at (197.0, 100.7)
- added TP11: BMS, TestPoint:TestPoint_Pad_D1.0mm, F.Cu at (203.2, 93.3)
- added TP12: LED, TestPoint:TestPoint_Pad_D1.0mm, F.Cu at (162.3, 85.2)
- added TP13: WK4, TestPoint:TestPoint_Pad_D1.0mm, F.Cu at (165.0, 84.8)
- added TP14: C2_1, TestPoint:TestPoint_Pad_D1.0mm, B.Cu at (168.7, 95.4)
- added TP15: C2_2, TestPoint:TestPoint_Pad_D1.0mm, B.Cu at (166.5, 95.4)
- added TP16: C3_1, TestPoint:TestPoint_Pad_D1.0mm, F.Cu at (173.1, 95.6)
- added TP17: TX, TestPoint:TestPoint_Pad_D1.0mm, F.Cu at (166.4, 98.3)
- added TP7: INT1, TestPoint:TestPoint_Pad_D1.0mm, B.Cu at (189.4, 89.4)
- added TP8: INT2, TestPoint:TestPoint_Pad_D1.0mm, B.Cu at (189.4, 91.4)
- added TP9: VCC, TestPoint:TestPoint_Pad_D1.0mm, F.Cu at (202.3, 100.7)
- C1: value 2u2 -> 10u
- C11: value 4p3 -> 1u
- C13: value 100n -> 4p3
- C3, C7: value 10u -> 100n
- C4: value 100n -> 10u
- C5, C6: value 1u -> 100n
- C8: value 100n -> 1u
- C9: value 100n -> 2u2
- R2: value 0 -> 10k
- R3: value 10k -> 0
- R5: value 100k -> 10k
- R6: value 10k -> 4k7
- R7: value 100k -> 4k7
- TP1: value SDA -> PB0
- TP2: value SCL -> PA7
- TP3: value INT1 -> PB1; moved to F.Cu
- TP4: value INT2 -> PA8; moved to F.Cu
- TP5: value VCC -> SDA
- TP6: value 3v -> SCL
- U1: value LIS2DW12 -> AP2205-3.0; footprint Package_LGA:LGA-12_2x2mm_P0.5mm -> Package_TO_SOT_SMD:SOT-23-5
- U2: value AP2205-3.0 -> BQ21080; footprint Package_TO_SOT_SMD:SOT-23-5 -> Components:Texas_DSBGA-8-1.04x1.59mm
- U3: value BQ21080 -> LIS2DW12; footprint Components:Texas_DSBGA-8-1.04x1.59mm -> Package_LGA:LGA-12_2x2mm_P0.5mm
- moved C7 39.4 mm to (163.6, 95.5), turned to 180 degrees
- moved C6 38.0 mm to (166.9, 85.5), turned to 180 degrees
- moved TP1 33.3 mm to (160.8, 92.5)
- moved TP2 33.3 mm to (160.4, 90.4)
- moved R4 29.9 mm to (173.7, 88.5), turned to -90 degrees
- moved TP3 28.8 mm to (161.2, 95.2), turned to 0 degrees
- moved R6 28.4 mm to (201.9, 92.2), turned to 0 degrees
- moved R7 26.2 mm to (201.0, 91.2), turned to 0 degrees
- moved TP4 26.1 mm to (164.2, 98.4), turned to 0 degrees
- moved R5 24.2 mm to (199.1, 94.9)
- moved C11 23.3 mm to (193.7, 78.4), turned to 90 degrees
- moved C8 23.1 mm to (202.8, 98.0)
- moved C5 23.0 mm to (172.3, 86.9), turned to 0 degrees
- moved C9 17.2 mm to (197.0, 98.2), turned to 90 degrees
- moved C15 16.6 mm to (180.0, 95.6), turned to 0 degrees
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Connections:
- C1 pad 1: +3V0 -> VCC
- C11 pad 1: GND -> +BATT
- C11 pad 2: Net-(U4-PC14) -> GND
- C12 pad 2: Net-(U4-PC15) -> Net-(U4-PC14)
- C13 pad 1: +3V0 -> GND
- C13 pad 2: GND -> Net-(U4-PC15)
- C14 pad 1: +3V0 -> ALVCC
- C15 pad 1: +3V0 -> ALVCC
- C2 pad 1: VCC -> VBUS
- C5 pad 1: +BATT -> +3V0
- C6 pad 1: VBUS -> +3V0
- C7 pad 1: VCC -> +3V0
- C8 pad 1: ALVCC -> VCC
- C9 pad 1: ALVCC -> +3V0
- R1 pad 1: +3V0 -> ~{BMS_INT}
- R1 pad 2: Net-(U1-~{CS}) -> +3V0
- R2 pad 1: GND -> +3V0
- R2 pad 2: Net-(U1-SA0/SDO) -> Net-(U3-~{CS})
- R3 pad 2: TS|MR -> Net-(U3-SA0/SDO)
- R4 pad 1: ~{BMS_INT} -> GND
- R4 pad 2: +3V0 -> Net-(U4-PH3)
- R5 pad 1: +3V0 -> GND
- R5 pad 2: BH1730PowerCtrl -> TS|MR
- R6 pad 1: GND -> SCL
- R6 pad 2: Net-(U4-PH3) -> +3V0
- R7 pad 1: +BATT -> SDA
- R7 pad 2: LEDPowerCtrl -> +3V0
- TP1 pad 1: SDA -> Net-(U4-PB0)
- TP2 pad 1: SCL -> Net-(U4-PA7)
- TP3 pad 1: IMU_INT1 -> Net-(U4-PB1)
- TP4 pad 1: IMU_INT2 -> Net-(U4-PA8)
- TP5 pad 1: VCC -> SDA
- TP6 pad 1: +3V0 -> SCL
- U1 pad 1: SCL -> VCC
- U1 pad 2: Net-(U1-~{CS}) -> GND
- U1 pad 3: Net-(U1-SA0/SDO) -> VCC
- U1 pad 4: SDA -> unconnected-(U1-NC-Pad4)
- U1 pad 5: GND -> +3V0
- U4 pad 13: unconnected-(U4-PA7-Pad13) -> Net-(U4-PA7)
- U4 pad 14: unconnected-(U4-PB0-Pad14) -> Net-(U4-PB0)
- U4 pad 15: unconnected-(U4-PB1-Pad15) -> Net-(U4-PB1)
- U4 pad 18: unconnected-(U4-PA8-Pad18) -> Net-(U4-PA8)
- U4 pad 25: BH1730PowerCtrl -> TSC_G3_IO1
- U4 pad 26: unconnected-(U4-PB3-Pad26) -> BH1730PowerCtrl
- U4 pad 27: unconnected-(U4-PB4-Pad27) -> TSC_G2_IO1
- U4 pad 28: unconnected-(U4-PB5-Pad28) -> TSC_G2_IO2
- U4 pad 8: unconnected-(U4-PA2-Pad8) -> WKUP4
Routing:
- net TSC_G2_IO2: track 0.00 -> 7.76 mm, vias 0 -> 1
- net TSC_G2_IO1: track 0.00 -> 5.42 mm, vias 0 -> 1
- net +3V0: track 78.2 -> 83.6 mm, vias 5 -> 6
- net Net-(U3-~{CS}): track 0.00 -> 3.89 mm, vias 0 -> 2
- net Net-(U1-~{CS}): track 3.89 -> 0.00 mm, vias 2 -> 0
- net Net-(U4-PA7): track 0.00 -> 3.82 mm
- net Net-(U4-PA8): track 0.00 -> 3.77 mm
- net Net-(U4-PB1): track 0.00 -> 3.44 mm
- net Net-(U3-SA0/SDO): track 0.00 -> 3.30 mm, vias 0 -> 2
- net Net-(U1-SA0/SDO): track 3.30 -> 0.00 mm, vias 2 -> 0
- net RX: track 0.00 -> 3.09 mm
- net TX: track 0.00 -> 3.08 mm
- net Net-(U4-PB0): track 0.00 -> 2.99 mm
- net (no net): track 172.3 -> 174.9 mm
- net WKUP4: track 0.00 -> 2.21 mm
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Other:
- board text added: "CLK"
- board text added: "DIO"
- board text added: "GND"
- board text added: "VBUS"
