File: mainboard.kicad_sch (KiCad schematic)
At the start: 27 parts, among them U1 LIS2DW12, U2 AP2205-3.0, U3 BQ21080, U4 STM32L412KBTx

Commit message: Diode layout, majority of schema, tile thoughts
Parts:
- added C10, C8, C9: 100n, Capacitor_SMD:C_0402_1005Metric, symbol Device:C_Small
- added C11, C12: 4p3, Capacitor_SMD:C_0402_1005Metric, symbol Device:C_Small
- added D1, D10, D11, D12, D13, D14, D15, D16, D2, D3, D4, D5, D6, D7, D8, D9: WS2812, LED_SMD:LED_WS2812_PLCC6_5.0x5.0mm_P1.6mm, symbol LED:WS2812
- added Q1, Q2: PMOS, Package_TO_SOT_SMD:SOT-23-3, symbol Simulation_SPICE:PMOS
- added R5, R7: 100k, Resistor_SMD:R_0402_1005Metric, symbol Device:R_Small
- added R6: 10k, Resistor_SMD:R_0402_1005Metric, symbol Device:R
- added U5: BH1730, symbol Components:BH1730
- added Y1: 32.768k, Crystal:Crystal_SMD_5032-2Pin_5.0x3.2mm, symbol Device:Crystal
Connections:
- net +3V0: now also C8.1, C9.1, Q1.3 (S), Q2.3 (S), R5.1, R7.1
- net GND: now also C10.1, C11.1, C12.1, C8.2, C9.2, D1.6 (VSS), D10.6 (VSS), D11.6 (VSS), D12.6 (VSS), D13.6 (VSS), D14.6 (VSS), D15.6 (VSS), D16.6 (VSS), D2.6 (VSS), D3.6 (VSS), D4.6 (VSS), D5.6 (VSS), D6.6 (VSS), D7.6 (VSS), D8.6 (VSS), D9.6 (VSS), R6.1, U5.2 (INT), U5.3 (GND)
- net IMU_INT1: now also U4.6 (PA0)
- net SCL: now also U4.29 (PB6), U5.6 (SCL)
- net SDA: now also U4.30 (PB7), U5.4 (SDA)
- net SWCLK: now also U4.24 (PA14)
- net SWDIO: now also U4.23 (PA13)
- net LED IN: now reaches U4.10 (PA4)
- net LED IN: now also D1.2 (DIN)
- net LEDPowerCtrl: now reaches U4.12 (PA6)
- net BH1730PowerCtrl: now reaches U4.13 (PA7)
- net BH1730PowerCtrl: now also Q1.2 (G), R5.2
- net TX: now reaches U4.19 (PA9)
- net at U4.2 (PC14): now also C11.2, Y1.2
- net RX: now reaches U4.20 (PA10)
- net at U4.3 (PC15): now also C12.2, Y1.1
- net at U4.31 (PH3): now also R6.2
- net at U4.4 (NRST): now also C10.2
- new net: D12.1 (DOUT), D13.2 (DIN)
- new net: D11.1 (DOUT), D12.2 (DIN)
- new net: D1.3 (VCC), D1.5 (VDD), D10.3 (VCC), D10.5 (VDD), D11.3 (VCC), D11.5 (VDD), D12.3 (VCC), D12.5 (VDD), D13.3 (VCC), D13.5 (VDD), D14.3 (VCC), D14.5 (VDD), D15.3 (VCC), D15.5 (VDD), D16.3 (VCC), D16.5 (VDD), D2.3 (VCC), D2.5 (VDD), D3.3 (VCC), D3.5 (VDD), D4.3 (VCC), D4.5 (VDD), D5.3 (VCC), D5.5 (VDD), D6.3 (VCC), D6.5 (VDD), D7.3 (VCC), D7.5 (VDD), D8.3 (VCC), D8.5 (VDD), D9.3 (VCC), D9.5 (VDD), Q2.1 (D)
- new net: D3.1 (DOUT), D4.2 (DIN)
- new net: D2.1 (DOUT), D3.2 (DIN)
- new net: D14.1 (DOUT), D15.2 (DIN)
- new net: D13.1 (DOUT), D14.2 (DIN)
- new net: D5.1 (DOUT), D6.2 (DIN)
- new net: D4.1 (DOUT), D5.2 (DIN)
- new net: D10.1 (DOUT), D11.2 (DIN)
- new net: D10.2 (DIN), D9.1 (DOUT)
- new net: D8.1 (DOUT), D9.2 (DIN)
- new net: D7.1 (DOUT), D8.2 (DIN)
- new net: Q1.1 (D), U5.1 (VCC), U5.5 (DVI)
- new net: D1.1 (DOUT), D2.2 (DIN)
- new net: D6.1 (DOUT), D7.2 (DIN)
- new net: D15.1 (DOUT), D16.2 (DIN)
- new net LEDP0werCtrl: Q2.2 (G), R7.2
Other:
- note added: "Light Sensor"
- moved on the sheet: U4

Commit message: Rev A layout. pending review
Parts:
- removed D1, D10, D11, D12, D13, D14, D15, D16, D2, D3, D4, D5, D6, D7, D8, D9: WS2812, LED_SMD:LED_WS2812_PLCC6_5.0x5.0mm_P1.6mm, symbol LED:WS2812
- removed Q1, Q2: PMOS, Package_TO_SOT_SMD:SOT-23-3, symbol Simulation_SPICE:PMOS
- removed TP10: DIO, TestPoint:TestPoint_Pad_D1.0mm, symbol Connector:TestPoint
- removed TP11: VBUS, TestPoint:TestPoint_Pad_D1.0mm, symbol Connector:TestPoint
- removed TP8: GND, TestPoint:TestPoint_Pad_D1.0mm, symbol Connector:TestPoint
- removed TP9: CLK, TestPoint:TestPoint_Pad_D1.0mm, symbol Connector:TestPoint
- added C13, C14, C15: 100n, Capacitor_SMD:C_0402_1005Metric, symbol Device:C_Small
- added J1: Conn_01x04_Pin, Connector_PinHeader_2.54mm:PinHeader_1x04_P2.54mm_Vertical, symbol Connector:Conn_01x04_Pin
- added Q2, Q3: Q_PMOS_GSD, Package_TO_SOT_SMD:SOT-23, symbol Device:Q_PMOS_GSD
- BT1: footprint (none) -> Components:battery_20x30
- U5: footprint (none) -> Components:WSOF6
- Y1: footprint Crystal:Crystal_SMD_5032-2Pin_5.0x3.2mm -> Crystal:Crystal_SMD_3215-2Pin_3.2x1.5mm
Connections:
- net LEDP0werCtrl is gone; now on net LEDPowerCtrl: R7.2
- net +3V0: now also C13.1, C14.1, C15.1, Q3.2 (S); no longer C8.1, C9.1, R7.1
- net +BATT: now also R7.1, Q2.2 (S)
- net BH1730PowerCtrl: now also U4.25 (PA15), Q3.1 (G); no longer U4.13 (PA7)
- net GND: now also C13.2, C14.2, C15.2, J1.1 (Pin_1)
- net LEDPowerCtrl: now also Q2.1 (G)
- net SWCLK: now also J1.2 (Pin_2)
- net SWDIO: now also J1.3 (Pin_3)
- net VBUS: now also J1.4 (Pin_4)
- net ALVCC: now reaches U5.1 (VCC), U5.5 (DVI)
- net ALVCC: now also C8.1, C9.1, Q3.3 (D)
- new net LED_PWR: Q2.3 (D)
Other:
- moved on the sheet: U4

Commit message: Rev 0 layout complete. ORdering as protoptype.
Parts:
- removed TP7: GND, TestPoint:TestPoint_Pad_D1.0mm, symbol Connector:TestPoint
- added R6, R7: 4k7, Resistor_SMD:R_0402_1005Metric, symbol Device:R
- added RX1: RX, TestPoint:TestPoint_Pad_D1.0mm, symbol Connector:TestPoint
- added TP1: PB0, TestPoint:TestPoint_Pad_D1.0mm, symbol Connector:TestPoint
- added TP11: BMS, TestPoint:TestPoint_Pad_D1.0mm, symbol Connector:TestPoint
- added TP12: LED, TestPoint:TestPoint_Pad_D1.0mm, symbol Connector:TestPoint
- added TP13: WK4, TestPoint:TestPoint_Pad_D1.0mm, symbol Connector:TestPoint
- added TP14: C2_1, TestPoint:TestPoint_Pad_D1.0mm, symbol Connector:TestPoint
- added TP15: C2_2, TestPoint:TestPoint_Pad_D1.0mm, symbol Connector:TestPoint
- added TP16: C3_1, TestPoint:TestPoint_Pad_D1.0mm, symbol Connector:TestPoint
- added TP17: TX, TestPoint:TestPoint_Pad_D1.0mm, symbol Connector:TestPoint
- added TP2: PA7, TestPoint:TestPoint_Pad_D1.0mm, symbol Connector:TestPoint
- added TP3: PB1, TestPoint:TestPoint_Pad_D1.0mm, symbol Connector:TestPoint
- added TP4: PA8, TestPoint:TestPoint_Pad_D1.0mm, symbol Connector:TestPoint
- C14: renamed from C9; now not fitted
- C15: renamed from C8; now not fitted
- Q1: renamed from Q3; now not fitted
- R8: renamed from R5; now not fitted
- U5: now not fitted
- renumbered C7 to C1, C5 to C11, C11 to C12, C12 to C13, C6 to C2, C4 to C3, C3 to C4, C13 to C5, C14 to C6, C15 to C7, C2 to C8, C1 to C9, R4 to R1, R1 to R2, R2 to R3, R6 to R4, R3 to R5, R7 to R9, TP6 to TP10, TP1 to TP5, TP2 to TP6, TP3 to TP7, TP4 to TP8, TP5 to TP9, U2 to U1, U3 to U2, U1 to U3
Connections:
- net +3V0: now also R6.2, R7.2
- net BH1730PowerCtrl: now also U4.26 (PB3); no longer U4.25 (PA15)
- net GND: no longer U1.3 (EN)
- net LED IN: now also TP12.1
- net RX: now also RX1.1
- net SCL: now also R6.1
- net SDA: now also R7.1
- net TX: now also TP17.1
- net VCC: now also U1.3 (EN)
- net ~{BMS_INT}: now also TP11.1
- net at U4.13 (PA7): now also TP2.1
- net at U4.14 (PB0): now also TP1.1
- net at U4.15 (PB1): now also TP3.1
- net at U4.18 (PA8): now also TP4.1
- net TSC_G2_IO1: now reaches U4.27 (PB4)
- net TSC_G2_IO1: now also TP14.1
- net TSC_G2_IO2: now reaches U4.28 (PB5)
- net TSC_G2_IO2: now also TP15.1
- net WKUP4: now reaches U4.8 (PA2)
- net WKUP4: now also TP13.1
- new net TSC_G3_IO1: TP16.1, U4.25 (PA15)
Other:
- note added: "in case needed"
- moved on the sheet: Q2
