File: BaseStation/BaseStation/BaseStation.kicad_pcb (KiCad board)
At the start: 2 copper layers, 18 parts, among them J1 USB_C_Receptacle_USB2.0_16P, J2 Conn_01x01_Pin, J3 Conn_01x01_Pin, J4 Conn_01x01_Pin, J5 Conn_01x01_Pin, SW1 SW_Push, U1 STM32F103CBTx, Y1 8M

Commit message: Somewhere around the first complete prototype. time to change BMS
Parts:
- removed the REF** at (157.0, 68.1)
- removed Y1: 8M, Crystal:Resonator_SMD-3Pin_7.2x3.0mm
- added C5: 100n, Capacitor_SMD:C_0402_1005Metric, F.Cu at (67.4, 87.9)
- added C6: 100n, Capacitor_SMD:C_0402_1005Metric, F.Cu at (58.4, 87.3)
- added C7: 100n, Capacitor_SMD:C_0402_1005Metric, F.Cu at (69.3, 80.8)
- added C8: 100n, Capacitor_SMD:C_0402_1005Metric, F.Cu at (61.1, 77.9)
- added C9: 100n, Capacitor_SMD:C_0402_1005Metric, F.Cu at (66.5, 77.9)
- added D1: LED, LED_SMD:LED_0603_1608Metric, F.Cu at (76.2, 80.1)
- added D2: D, Diode_SMD:D_SOD-323, F.Cu at (77.7, 90.4)
- added J10: Conn_01x04_Pin, Connector_PinHeader_2.54mm:PinHeader_1x04_P2.54mm_Horizontal, F.Cu at (82.4, 70.8)
- added J6: Conn_01x01_Pin, TestPoint:TestPoint_Pad_D1.5mm, F.Cu at (61.0, 70.4)
- added J7: Conn_01x01_Pin, TestPoint:TestPoint_Pad_D1.5mm, F.Cu at (62.2, 68.2)
- added J8: Conn_01x01_Pin, TestPoint:TestPoint_Pad_D1.5mm, F.Cu at (63.5, 66.0)
- added J9: Conn_01x01_Pin, TestPoint:TestPoint_Pad_D1.5mm, F.Cu at (64.8, 63.8)
- added Q1: Q_PNP_BEC, Package_TO_SOT_SMD:SOT-23, F.Cu at (81.3, 91.4)
- added Q3: Q_NPN_BEC, Package_TO_SOT_SMD:SOT-23, F.Cu at (86.1, 91.4)
- added R10: 330r, Resistor_SMD:R_0402_1005Metric, F.Cu at (77.7, 91.9)
- added R6: 510r, Resistor_SMD:R_0603_1608Metric, F.Cu at (76.2, 81.8)
- added R7: 1k, Resistor_SMD:R_0402_1005Metric, F.Cu at (83.8, 93.0)
- added R8: 330r, Resistor_SMD:R_0402_1005Metric, F.Cu at (83.8, 89.9)
- added R9: 10k, Resistor_SMD:R_0402_1005Metric, F.Cu at (82.5, 88.6)
- added REF**: MountingHole_2.2mm_M2, MountingHole:MountingHole_2.2mm_M2, F.Cu at (98.1, 92.8)
- added REF**: MountingHole_2.2mm_M2, MountingHole:MountingHole_2.2mm_M2, F.Cu at (54.3, 92.8)
- added REF**: MountingHole_2.2mm_M2, MountingHole:MountingHole_2.2mm_M2, F.Cu at (76.2, 54.9)
- added U2: AMS1117-3.3, Package_TO_SOT_SMD:SOT-223-3_TabPin2, F.Cu at (93.5, 82.8)
- added Y2: 8M, Crystal:Crystal_SMD_5032-2Pin_5.0x3.2mm, F.Cu at (63.8, 75.2)
- C3, C4: footprint Capacitor_SMD:C_0603_1608Metric -> Capacitor_SMD:C_0402_1005Metric
- J2, J3, J4, J5: footprint Connector_PinHeader_2.00mm:PinHeader_1x01_P2.00mm_Horizontal -> TestPoint:TestPoint_Loop_D3.50mm_Drill0.9mm_Beaded
- moved C4 110.7 mm to (62.7, 72.6), turned to 180 degrees
- moved R4 109.1 mm to (56.1, 84.3), turned to 0 degrees
- moved R3 108.8 mm to (58.6, 77.6)
- moved C3 108.0 mm to (64.8, 72.6)
- moved U1 104.1 mm to (63.2, 83.6), turned to -90 degrees
- moved R1 98.0 mm to (69.8, 97.5), turned to -90 degrees
- moved R5 96.5 mm to (73.9, 66.4), turned to 180 degrees
- moved J2 93.3 mm to (79.6, 87.3), turned to 0 degrees
- moved J3 91.5 mm to (77.3, 87.3), turned to 0 degrees
- moved SW1 90.0 mm to (76.2, 62.7), turned to 0 degrees
- moved J4 89.8 mm to (75.1, 87.3), turned to 0 degrees
- moved J5 88.0 mm to (72.8, 87.3), turned to 0 degrees
- moved J1 87.3 mm to (76.2, 98.6), turned to 0 degrees
- moved R2 82.5 mm to (82.5, 97.5), turned to -90 degrees
- moved C1 67.7 mm to (89.4, 87.9), turned to -150 degrees
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Connections:
- J2 pad 1: VBUS -> VCHRG
- U1 pad 15: unconnected-(U1-PA5-Pad15) -> SWSCK
- U1 pad 2: unconnected-(U1-PC13-Pad2) -> Net-(U1-PC13)
- U1 pad 28: unconnected-(U1-PB15-Pad28) -> SWDIO
- U1 pad 34: SWDIO -> SWDIO_DBG
- U1 pad 37: SWSCK -> SWSCK_DBG
Routing:
- net +3V3: track 0.00 -> 98.1 mm
- net VBUS: track 0.00 -> 51.0 mm, vias 0 -> 2
- net SWDIO: track 0.00 -> 36.6 mm, vias 0 -> 3
- net SWSCK: track 0.00 -> 34.6 mm, vias 0 -> 1
- net SWSCK_DBG: track 0.00 -> 27.9 mm, vias 0 -> 2
- net SWDIO_DBG: track 0.00 -> 25.9 mm, vias 0 -> 2
- net USB_D+: track 0.00 -> 19.3 mm
- net USB_D-: track 0.00 -> 19.3 mm
- net BOOT0: track 9.29 -> 28.2 mm, vias 0 -> 2
- net Net-(U1-PC13): track 0.00 -> 11.7 mm, vias 0 -> 2
- net Net-(J1-CC2): track 0.00 -> 11.5 mm, vias 0 -> 2
- net VCHRG: track 0.00 -> 9.97 mm
- net Net-(J1-CC1): track 0.00 -> 9.72 mm
- net GND: track 0.00 -> 5.77 mm, vias 0 -> 36
- net Net-(U1-NRST): track 10.4 -> 5.66 mm, vias 2 -> 0
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- added copper zone on B.Cu, net GND
- added copper zone on F.Cu, net GND
Other:
- board outline added: 52.1 x 49 mm
- board text added: "+3v3"
- board text added: "CLK"
- board text added: "DIO"
- board text added: "EEAN"
- board text added: "GND"
- board text added: "JLCJLCJLCJLC"
- board text added: "Rev. A"
