File: BaseStation/BaseStation/BaseStation.kicad_sch (KiCad schematic)
At the start: 18 parts, among them J1 USB_C_Receptacle_USB2.0_16P, J2 Conn_01x01_Pin, J3 Conn_01x01_Pin, J4 Conn_01x01_Pin, J5 Conn_01x01_Pin, SW1 SW_Push, U1 STM32F103CBTx, U2 AMS1117-3.3, Y1 8M

Commit message: Somewhere around the first complete prototype. time to change BMS
Parts:
- removed Y1: 8M, Crystal:Resonator_SMD-3Pin_7.2x3.0mm, symbol Device:Crystal_GND2
- added C5, C6, C7, C8, C9: 100n, Capacitor_SMD:C_0402_1005Metric, symbol Device:C_Small
- added D1: LED, LED_SMD:LED_0603_1608Metric, symbol Device:LED
- added D2: D, Diode_SMD:D_SOD-323, symbol Device:D
- added J10: Conn_01x04_Pin, Connector_PinHeader_2.54mm:PinHeader_1x04_P2.54mm_Horizontal, symbol Connector:Conn_01x04_Pin
- added J6, J7, J8, J9: Conn_01x01_Pin, TestPoint:TestPoint_Pad_D1.5mm, symbol Connector:Conn_01x01_Pin
- added Q1: Q_PNP_BEC, Package_TO_SOT_SMD:SOT-23, symbol Device:Q_PNP_BEC
- added Q3: Q_NPN_BEC, Package_TO_SOT_SMD:SOT-23, symbol Device:Q_NPN_BEC
- added R10, R8: 330r, Resistor_SMD:R_0402_1005Metric, symbol Device:R
- added R11: 1k5, Resistor_SMD:R_0402_1005Metric, symbol Device:R
- added R6: 510r, Resistor_SMD:R_0603_1608Metric, symbol Device:R
- added R7: 1k, Resistor_SMD:R_0402_1005Metric, symbol Device:R
- added R9: 10k, Resistor_SMD:R_0402_1005Metric, symbol Device:R
- added Y2: 8M, Crystal:Crystal_SMD_5032-2Pin_5.0x3.2mm, symbol Device:Crystal
- C3, C4: footprint Capacitor_SMD:C_0603_1608Metric -> Capacitor_SMD:C_0402_1005Metric
- J2, J3, J4, J5: footprint Connector_PinHeader_2.00mm:PinHeader_1x01_P2.00mm_Horizontal -> TestPoint:TestPoint_Loop_D3.50mm_Drill0.9mm_Beaded
Connections:
- net +3V3: now also C5.1, C6.1, C7.1, C8.1, C9.1, D1.2 (A), J6.1 (Pin_1), R11.1
- net GND: now also C5.2, C6.2, C7.2, C8.2, C9.2, J10.4 (Pin_4), J9.1 (Pin_1), Q3.2 (E), R9.2
- net SWDIO: now also U1.27 (PB14), J10.2 (Pin_2); no longer U1.34 (PA13)
- net SWSCK: now also U1.15 (PA5), J10.3 (Pin_3); no longer U1.37 (PA14)
- net USB_D+: now also R11.2
- net VBUS: now also J10.1 (Pin_1), Q1.3 (C), R10.1; no longer J2.1 (Pin_1)
- net at U1.2 (PC13): now also R6.2
- net at C3.2, U1.5 (PD0): now also Y2.2
- net at C4.2, U1.6 (PD1): now also Y2.1
- new net: Q1.1 (B), R7.1
- new net: D2.2 (A), R10.2
- new net: D1.1 (K), R6.1
- new net: Q3.1 (B), R8.1
- new net: Q3.3 (C), R7.2
- new net SWDIO_DBG: J7.1 (Pin_1), U1.34 (PA13)
- new net SWSCK_DBG: J8.1 (Pin_1), U1.37 (PA14)
- new net VCHRG: D2.1 (K), J2.1 (Pin_1), Q1.2 (E), R8.2, R9.1
Other:
- note added: "3v3 Regulator"
- note added: "DBG PRG"
- note added: "EXT PROG"
- note added: "Functionally an STM32 BluePill based on STM32F103CBT6. Flashed as a blackmagic probe. Target 100% Assembly by JLC Target 100% "basic" parts - STM32F103 is not - Pogo Pins are not. - The rest should be."
- note added: "POGO Pins"
- note added: "PROGRAMMING"
- note added: "Short Circuit Protection"
- note added: "USB"
- note added: "https://medium.com/@paramaggarwal/converting-an-stm32f103-board-to-a-black-magic-probe-c013cf2cc38c"
- moved on the sheet: U1
