File: Mainboard/bms.kicad_sch (KiCad schematic)
At the start: 12 parts, among them IC1 TLV3691IDPFR, J2 Conn_01x02_Socket, J3 Conn_01x02_Socket, Q1 Q_PMOS_GSD, U2 TPS7A0218PDBVR, U5 MCP73832-2-OT

Commit message: V2 mainboard, some firmware stuffs, free design files I guess
Parts:
- removed IC1: TLV3691IDPFR, TLV3691IDPFR, symbol TLV3691IDPFR:TLV3691IDPFR
- removed Q1: Q_PMOS_GSD, Package_TO_SOT_SMD:SOT-23, symbol Device:Q_PMOS_GSD
- removed R1: 10M, Resistor_SMD:R_0402_1005Metric, symbol Device:R_Small
- removed R11: 2M, Resistor_SMD:R_0402_1005Metric, symbol Device:R
- removed R5: 1M8, Resistor_SMD:R_0402_1005Metric, symbol Device:R
- removed U2: TPS7A0218PDBVR, Package_TO_SOT_SMD:SOT-23-5, symbol Regulator_Linear:TPS7A0518PDBV
- added D34: D, Diode_SMD:D_SOD-323, symbol Device:D
- added Q3: Q_PMOS_GSD, Package_TO_SOT_SMD:SOT-23, symbol Device:Q_PMOS_GSD
- added R15: 100k, Resistor_SMD:R_0402_1005Metric, symbol Device:R
Connections:
- net +BATT: now also Q3.3 (D)
- net GND: now also R15.1
- net VBUS: now also D34.2 (A), Q3.1 (G), R15.2
- net VCC: now also D34.1 (K), Q3.2 (S)
Other:
- note added: "Power Path Regulation Adds a ~0.5v drop to batt. Somehow this still drives the LEDs."
- note removed: "Undervoltage Protection"
